File: Hardware/LongWaveModule.brd (EAGLE design)
At the start: 39.4 x 16.9 mm, 41 parts, among them J1 CONN_42.54_SCREW, Q1 2N7002, Q2 2N7002, Q3 DMG3404, U1 STP-135SR, U2 LTC2050HV, U3 LTC2054, U4 LTC2054, U5 TPS60403, U6 TPS79733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

Commit message: Dyson --> Monarch in sch and on silk
Other:
- board text added: "Project Monarch v0.1 LongWave ---------------- Developed by Northern Widget and University of Minnesota"
- board text removed: "Project Dyson v0.1 LongWave ---------------- Developed by Northern Widget and University of Minnesota"
Changed lines of the file:
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@@
 <?xml version="1.0" encoding="utf-8"?>
 <!DOCTYPE eagle SYSTEM "eagle.dtd">
-<eagle version="9.2.1">
+<eagle version="9.6.2">
 <drawing>
 <settings>
-<setting alwaysvectorfont="no"/>
+<setting alwaysvectorfont="yes"/>
 <setting verticaltext="up"/>
 </settings>
@@
 <text x="8.509" y="1.905" size="0.8128" layer="52" font="vector" ratio="15" rot="SMR270" align="center">ADR
 Select</text>
-<text x="17.145" y="12.827" size="0.8128" layer="52" font="vector" ratio="15" rot="MR0" align="center-left">Project Dyson v0.1
+<text x="17.145" y="12.827" size="0.8128" layer="52" font="vector" ratio="15" rot="MR0" align="center-left">Project Monarch v0.1
 LongWave
 ----------------
