File: Hardware/LongWaveModule.sch (EAGLE design)
At the start: 41 parts, among them J1 CONN_42.54_SCREW, Q2 DMG3404, Q4 2N7002, Q5 2N7002

Commit message: Made fixes to #2, #3, #4
Fixed the silk screen numbering issue, fixed pinout of thermopile, connected voltage ref pin
Connections:
- removed net N$10: C12.2, U$9.GND
- net GND: now also C12.2, U$9.GND
Changed lines of the file:
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@@
 <?xml version="1.0" encoding="utf-8"?>
 <!DOCTYPE eagle SYSTEM "eagle.dtd">
-<eagle version="8.5.1">
+<eagle version="9.0.1">
 <drawing>
 <settings>
@@
 <part name="H2" library="bschulz" deviceset="MOUNTING_HOLE" device="2_NP" value="2-56"/>
 <part name="H3" library="bschulz" deviceset="MOUNTING_HOLE" device="2_NP" value="2-56"/>
+<part name="GND5" library="supply1" library_urn="urn:adsk.eagle:library:371" deviceset="GND" device=""/>
 </parts>
 <sheets>
@@
 <instance part="H2" gate="G$1" x="243.84" y="53.34"/>
 <instance part="H3" gate="G$1" x="243.84" y="48.26"/>
+<instance part="GND5" gate="1" x="261.62" y="73.66"/>
 </instances>
 <busses>
@@
 <wire x1="195.58" y1="121.92" x2="195.58" y2="124.46" width="0.1524" layer="91"/>
 </segment>
+<segment>
+<pinref part="U$9" gate="G$1" pin="GND"/>
+<pinref part="C12" gate="G$1" pin="2"/>
+<wire x1="256.54" y1="78.74" x2="261.62" y2="78.74" width="0.1524" layer="91"/>
+<pinref part="GND5" gate="1" pin="GND"/>
+<wire x1="261.62" y1="76.2" x2="261.62" y2="78.74" width="0.1524" layer="91"/>
+<junction x="261.62" y="78.74"/>
+</segment>
 </net>
 <net name="N$1" class="0">
@@
 </segment>
 </net>
-<net name="N$10" class="0">
-<segment>
-<pinref part="U$9" gate="G$1" pin="GND"/>
-<pinref part="C12" gate="G$1" pin="2"/>
-<wire x1="256.54" y1="78.74" x2="261.62" y2="78.74" width="0.1524" layer="91"/>
-</segment>
-</net>

Commit message: Updated part info, license and BOM
Parts:
- removed C14, C15, C16, C17, C18: 1uF, bschulz_passives:C-EUC0603
- removed Q5: 2N7002, bschulz:MOSFET-NCH-2N7002PW
- removed R13, R14, R15, R16: 10k, bschulz_passives:R-EU_R0603
- removed U$4, U$5: LTC2054HV, bschulz:LTC2054HV
- added C5, C6, C9: 0.1uF, bschulz_passives:C-EU0.1UFC0603
- added C7, C8: 1uF, bschulz_passives:C-EU1UFC0603
- added Q3: DMG3404, bschulz:MOSFET-NCH-DMG3404L
- added R10, R11: 100k, bschulz_passives:R-EU_P100KR0603
- added R12: 1k, bschulz_passives:R-EU_1KR0603
- added R9: 1k, bschulz_passives:R-EU_P1KR0603
- added U3, U4: LTC2050HV, bschulz:LTC2050HV
- C1, C2, C3, C4: value 0.1uF -> 1uF; device bschulz_passives:C-EUC0603 -> bschulz_passives:C-EU1UFC0603
- C10, C11, C12: device bschulz_passives:C-EUC0603 -> bschulz_passives:C-EU0.1UFC0603
- C13: value 1uF -> 0.1uF; device bschulz_passives:C-EUC0603 -> bschulz_passives:C-EU0.1UFC0603
- Q2: value DMG3404 -> 2N7002; device bschulz:MOSFET-NCH-DMG3404L -> bschulz:MOSFET-NCH-2N7002PW
- R1, R2: value 1k -> 10k; device bschulz_passives:R-EU_R0603 -> bschulz_passives:R-EU_10KR0603
- R3: value 100k -> 10k; device bschulz_passives:R-EU_R0603 -> bschulz_passives:R-EU_P10KR0603
- R4, R5: value 100k -> 10k; device bschulz_passives:R-EU_R0603 -> bschulz_passives:R-EU_10KR0603
- R6: device bschulz_passives:R-EU_R0603 -> bschulz_passives:R-EU_P100KR0603
- R7: value 10k -> 100k; device bschulz_passives:R-EU_R0603 -> bschulz_passives:R-EU_P100KR0603
- R8: device bschulz_passives:R-EU_R0603 -> bschulz_passives:R-EU_P1KR0603
- renumbered Q4 to Q1, U$1 to U1, U$10 to U5, U$11 to U6, U$2 to U7, U$3 to U2, U$9 to U8
Connections:
- net -VCC: now also C5.2, C7.1, R12.2; no longer C1.2, C18.1, R8.2
- net AOUT_THERMISTOR: now also R3.1; no longer R7.1
- net AOUT_THERMOPILE: now also R11.1, U4.OUT; no longer R3.1, U$5.OUT
- net GND: now also C1.2, C6.2, C7.2, C8.2, C9.2, Q3.S, R7.1, R9.1, U3.VSS, U4.VSS; no longer C14.2, C16.2, C17.2, C18.2, C2.2, Q2.S, R2.1, R6.1, U$4.VSS, U$5.VSS
- net N$1: now also R8.1; no longer R1.1
- net N$11: now also C2.1; no longer C15.1
- net N$12: now also C2.2; no longer C15.2
- net N$2: now also R10.2, R8.2, U4.VIN+; no longer R1.2, R4.2, U$5.VIN+
- net N$21: now also C4.1, R12.1; no longer C14.1, R8.1
- net N$3: now also R11.2, R9.2, U4.VIN-; no longer R2.2, R3.2, U$5.VIN-
- net N$5: now also R10.1, U3.OUT, U3.VIN-; no longer R4.1, U$4.OUT, U$4.VIN-
- net N$6: now also R6.1, R7.2, U3.VIN+; no longer R5.1, R6.2, U$4.VIN+
- net N$8: now also C12.1; no longer C11.1
- net SCL: now also Q2.S, R2.1; no longer Q5.S, R14.1
- net SCL_EXT: now also Q2.D, R5.1; no longer Q5.D, R16.1
- net SDA: now also R1.1; no longer R13.1
- net SDA_EXT: now also R4.1; no longer R15.1
- net VCC: now also C11.1, C5.1, C6.1, C8.1, C9.1, Q2.G, R1.2, R2.2, U3.VDD, U4.VDD; no longer C13.1, C16.1, C2.1, C3.1, C4.1, Q5.G, R13.2, R14.2, U$4.VDD, U$5.VDD
- net VIN+: now also C3.1, Q3.G, R4.2, R5.2; no longer C17.1, Q2.G, R15.2, R16.2
- net VIN-: now also Q3.D; no longer Q2.D
- net VREF: now also C13.1, R3.2, R6.2; no longer C12.1, R5.2, R7.2
Other:
- moved on the sheet: C1, C10, C11, C12, C13, C2, C3, C4, Q2, R1, R2, R3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

Commit message: Generated gerbers for Mrk 0.1
Added Gerbers for Mrk 0.1 revision, fixed silk screen issues, added pullup resistors for on board I2C on shortwave module, and changed amplifiers on longwave module (eliminated use of LTC2054HV, and switched to using LTC2050HV due to availability), also fixed (flipped) thermistor arraignment on shortwave module
Parts:
- U2: value LTC2054HV -> LTC2050HV; device bschulz:LTC2054HV -> bschulz:LTC2050HV
- U3, U4: value LTC2050HV -> LTC2054; device bschulz:LTC2050HV -> bschulz:LTC2054
Changed lines of the file:
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@@
 <grid distance="0.1" unitdist="inch" unit="inch" style="lines" multiple="1" display="no" altdistance="0.01" altunitdist="inch" altunit="inch"/>
 <layers>
-<layer number="1" name="Top" color="4" fill="1" visible="yes" active="no"/>
-<layer number="2" name="Route2" color="1" fill="3" visible="yes" active="no"/>
-<layer number="3" name="Route3" color="4" fill="3" visible="yes" active="no"/>
-<layer number="4" name="Route4" color="1" fill="4" visible="yes" active="no"/>
-<layer number="5" name="Route5" color="4" fill="4" visible="yes" active="no"/>
-<layer number="6" name="Route6" color="1" fill="8" visible="yes" active="no"/>
-<layer number="7" name="Route7" color="4" fill="8" visible="yes" active="no"/>
-<layer number="8" name="Route8" color="1" fill="2" visible="yes" active="no"/>
-<layer number="9" name="Route9" color="4" fill="2" visible="yes" active="no"/>
-<layer number="10" name="Route10" color="1" fill="7" visible="yes" active="no"/>
-<layer number="11" name="Route11" color="4" fill="7" visible="yes" active="no"/>
-<layer number="12" name="Route12" color="1" fill="5" visible="yes" active="no"/>
-<layer number="13" name="Route13" color="4" fill="5" visible="yes" active="no"/>
-<layer number="14" name="Route14" color="1" fill="6" visible="yes" active="no"/>
-<layer number="15" name="Route15" color="4" fill="6" visible="yes" active="no"/>
-<layer number="16" name="Bottom" color="1" fill="1" visible="yes" active="no"/>
-<layer number="17" name="Pads" color="2" fill="1" visible="yes" active="no"/>
-<layer number="18" name="Vias" color="2" fill="1" visible="yes" active="no"/>
-<layer number="19" name="Unrouted" color="6" fill="1" visible="yes" active="no"/>
-<layer number="20" name="Dimension" color="24" fill="1" visible="yes" active="no"/>
-<layer number="21" name="tPlace" color="7" fill="1" visible="yes" active="no"/>
-<layer number="22" name="bPlace" color="7" fill="1" visible="yes" active="no"/>
-<layer number="23" name="tOrigins" color="15" fill="1" visible="yes" active="no"/>
-<layer number="24" name="bOrigins" color="15" fill="1" visible="yes" active="no"/>
-<layer number="25" name="tNames" color="7" fill="1" visible="yes" active="no"/>
-<layer number="26" name="bNames" color="7" fill="1" visible="yes" active="no"/>
-<layer number="27" name="tValues" color="7" fill="1" visible="yes" active="no"/>
-<layer number="28" name="bValues" color="7" fill="1" visible="yes" active="no"/>
+<layer number="1" name="Top" color="4" fill="1" visible="no" active="no"/>
+<layer number="2" name="Route2" color="1" fill="3" visible="no" active="no"/>
+<layer number="3" name="Route3" color="4" fill="3" visible="no" active="no"/>
+<layer number="4" name="Route4" color="1" fill="4" visible="no" active="no"/>
+<layer number="5" name="Route5" color="4" fill="4" visible="no" active="no"/>
+<layer number="6" name="Route6" color="1" fill="8" visible="no" active="no"/>
+<layer number="7" name="Route7" color="4" fill="8" visible="no" active="no"/>
+<layer number="8" name="Route8" color="1" fill="2" visible="no" active="no"/>
+<layer number="9" name="Route9" color="4" fill="2" visible="no" active="no"/>
+<layer number="10" name="Route10" color="1" fill="7" visible="no" active="no"/>
+<layer number="11" name="Route11" color="4" fill="7" visible="no" active="no"/>
+<layer number="12" name="Route12" color="1" fill="5" visible="no" active="no"/>
+<layer number="13" name="Route13" color="4" fill="5" visible="no" active="no"/>
+<layer number="14" name="Route14" color="1" fill="6" visible="no" active="no"/>
+<layer number="15" name="Route15" color="4" fill="6" visible="no" active="no"/>
+<layer number="16" name="Bottom" color="1" fill="1" visible="no" active="no"/>
+<layer number="17" name="Pads" color="2" fill="1" visible="no" active="no"/>
+<layer number="18" name="Vias" color="2" fill="1" visible="no" active="no"/>
+<layer number="19" name="Unrouted" color="6" fill="1" visible="no" active="no"/>
+<layer number="20" name="Dimension" color="24" fill="1" visible="no" active="no"/>
+<layer number="21" name="tPlace" color="7" fill="1" visible="no" active="no"/>
+<layer number="22" name="bPlace" color="7" fill="1" visible="no" active="no"/>
+<layer number="23" name="tOrigins" color="15" fill="1" visible="no" active="no"/>
+<layer number="24" name="bOrigins" color="15" fill="1" visible="no" active="no"/>
+<layer number="25" name="tNames" color="7" fill="1" visible="no" active="no"/>
+<layer number="26" name="bNames" color="7" fill="1" visible="no" active="no"/>
+<layer number="27" name="tValues" color="7" fill="1" visible="no" active="no"/>
+<layer number="28" name="bValues" color="7" fill="1" visible="no" active="no"/>
 <layer number="29" name="tStop" color="7" fill="3" visible="no" active="no"/>
 <layer number="30" name="bStop" color="7" fill="6" visible="no" active="no"/>
@@
 <layer number="35" name="tGlue" color="7" fill="4" visible="no" active="no"/>
 <layer number="36" name="bGlue" color="7" fill="5" visible="no" active="no"/>
-<layer number="37" name="tTest" color="7" fill="1" visible="yes" active="no"/>
-<layer number="38" name="bTest" color="7" fill="1" visible="yes" active="no"/>
+<layer number="37" name="tTest" color="7" fill="1" visible="no" active="no"/>
+<layer number="38" name="bTest" color="7" fill="1" visible="no" active="no"/>
 <layer number="39" name="tKeepout" color="4" fill="11" visible="no" active="no"/>
 <layer number="40" name="bKeepout" color="1" fill="11" visible="no" active="no"/>
@@
 <layer number="44" name="Drills" color="7" fill="1" visible="no" active="no"/>
 <layer number="45" name="Holes" color="7" fill="1" visible="no" active="no"/>
-<layer number="46" name="Milling" color="3" fill="1" visible="yes" active="no"/>
-<layer number="47" name="Measures" color="7" fill="1" visible="yes" active="no"/>
-<layer number="48" name="Document" color="7" fill="1" visible="yes" active="no"/>
-<layer number="49" name="Reference" color="7" fill="1" visible="yes" active="no"/>
-<layer number="50" name="dxf" color="7" fill="1" visible="yes" active="no"/>
-<layer number="51" name="tDocu" color="7" fill="1" visible="yes" active="no"/>
-<layer number="52" name="bDocu" color="7" fill="1" visible="yes" active="no"/>
-<layer number="53" name="tGND_GNDA" color="7" fill="1" visible="yes" active="no"/>
-<layer number="54" name="bGND_GNDA" color="7" fill="1" visible="yes" active="no"/>
-<layer number="56" name="wert" color="7" fill="1" visible="yes" active="no"/>
-<layer number="57" name="tCAD" color="7" fill="1" visible="yes" active="no"/>
-<layer number="59" name="tCarbon" color="7" fill="1" visible="yes" active="no"/>
-<layer number="60" name="bCarbon" color="7" fill="1" visible="yes" active="no"/>
+<layer number="46" name="Milling" color="3" fill="1" visible="no" active="no"/>
+<layer number="47" name="Measures" color="7" fill="1" visible="no" active="no"/>
+<layer number="48" name="Document" color="7" fill="1" visible="no" active="no"/>
+<layer number="49" name="Reference" color="7" fill="1" visible="no" active="no"/>
+<layer number="50" name="dxf" color="7" fill="1" visible="no" active="no"/>
+<layer number="51" name="tDocu" color="7" fill="1" visible="no" active="no"/>
+<layer number="52" name="bDocu" color="7" fill="1" visible="no" active="no"/>
+<layer number="53" name="tGND_GNDA" color="7" fill="1" visible="no" active="no"/>
+<layer number="54" name="bGND_GNDA" color="7" fill="1" visible="no" active="no"/>
+<layer number="56" name="wert" color="7" fill="1" visible="no" active="no"/>
+<layer number="57" name="tCAD" color="7" fill="1" visible="no" active="no"/>
+<layer number="59" name="tCarbon" color="7" fill="1" visible="no" active="no"/>
+<layer number="60" name="bCarbon" color="7" fill="1" visible="no" active="no"/>
 <layer number="88" name="SimResults" color="9" fill="1" visible="yes" active="yes"/>
 <layer number="89" name="SimProbes" color="9" fill="1" visible="yes" active="yes"/>
@@
 <part name="U1" library="bschulz" deviceset="STP-135SR" device=""/>
 <part name="U7" library="bschulz" deviceset="ADS111*" device="" technology="5"/>
-<part name="U2" library="bschulz" deviceset="LTC2054" device="" technology="HV"/>
-<part name="U3" library="bschulz" deviceset="LTC2050" device="" technology="HV"/>
-<part name="U4" library="bschulz" deviceset="LTC2050" device="" technology="HV"/>
+<part name="U2" library="bschulz" deviceset="LTC2050" device="" technology="HV"/>
+<part name="U3" library="bschulz" deviceset="LTC2054" device="" value="LTC2054"/>
+<part name="U4" library="bschulz" deviceset="LTC2054" device="" value="LTC2054"/>
 <part name="GND1" library="supply1" library_urn="urn:adsk.eagle:library:371" deviceset="GND" device=""/>
 <part name="R8" library="bschulz_passives" deviceset="R-EU_" device="R0603" technology="P1K" value="1k"/>
@@
 <attribute name="DESIGNER" value="Bobby Schulz"/>
 <attribute name="PROJECT" value="Dyson"/>
-<attribute name="REV" value="0.0"/>
+<attribute name="REV" value="0.1"/>
 </part>
 <part name="GND5" library="supply1" library_urn="urn:adsk.eagle:library:371" deviceset="GND" device=""/>
